File: WirelessQAZ.sch (KiCad schematic (older format))
At the start: 124 parts, among them J2 Switch, J3 BATT, J4 SWD, Q1 AO3400A, SW1 SW_Push, U1 nRF52840_holyiot_18010, U2 USBLC6-2SC6, U3 DW01A, U4 XC6206P332MR, U5 TP4056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

Commit message: re
Connections:
- wire segments 229 -> 232
Changed lines of the file:
@@
 $EndComp
 Wire Wire Line
-	7750 5150 6950 5150
+	7750 5150 7550 5150
 Wire Wire Line
 	6950 5150 6950 5200
@@
 Wire Wire Line
 	5000 2650 10150 2650
+Text HLabel 7750 4750 2    50   Input ~ 0
+5V_USB
+Wire Wire Line
+	7550 5250 7550 5150
+Connection ~ 7550 5150
+Wire Wire Line
+	7550 5150 6950 5150
+Wire Wire Line
+	7750 4750 7750 5150
+Connection ~ 7750 5150
 $EndSCHEMATC
