File: WirelessQAZ.kicad_pcb (KiCad board)
At the start: 2 copper layers, 189.3 x 78.1 mm, 124 parts, among them Q1 AO3400A, SW1 SW_Push, U1 nRF52840_holyiot_18010, U2 USBLC6-2SC6, U3 DW01A, U4 XC6206P332MR, U5 TP4056, U6 FS8205

Commit message: things happening
Other:
- net class Default removed
